Commit message: Reach working PoC

File: urdf/cartpole.xacro (robot description, xacro)
@@ -2,5 +2,5 @@
 <robot xmlns:xacro="http://www.ros.org/wiki/xacro" name="cartpole">
 	<!-- Properties -->
-	<xacro:property name="obj_scale" value="0.001" />
+	<xacro:property name="obj_scale" value="1.000" />
 	<!-- Define colors -->
 	<material name="black">
@@ -16,5 +16,5 @@
 		<origin rpy="0.0 0 0" xyz="0 0 0" />
 		<geometry>
-			<mesh filename="package://meshes/beam-Body.obj" scale="${obj_scale} ${obj_scale} ${obj_scale}" />
+			<mesh filename="$(find cartpole_01)/meshes/beam.dae" scale="${obj_scale} ${obj_scale} ${obj_scale}" />
 		</geometry>
 	</xacro:macro>
@@ -38,22 +38,24 @@
 	</link>
 	<gazebo reference="beam">
-		<mu1>
+		<!-- <mu1>
 			0.2
 		</mu1>
 		<mu2>
 			0.2
-		</mu2>
-		<!-- Chrome: http://www.barradeau.com/nicoptere/dump/materials.html -->
-		<material>
-			<diffuse>
-				0.4 0.4 0.4 1
-			</diffuse>
-			<ambient>
-				0.25 0.25 0.25 1
-			</ambient>
-			<specular>
-				0.774597 0.774597 0.774597 1
-			</specular>
-		</material>
+		</mu2> -->
+		<visual>
+			<!-- Chrome: http://www.barradeau.com/nicoptere/dump/materials.html -->
+			<material>
+				<diffuse>
+					0.4 0.4 0.4 1
+				</diffuse>
+				<ambient>
+					0.25 0.25 0.25 1
+				</ambient>
+				<specular>
+					0.774597 0.774597 0.774597 1
+				</specular>
+			</material>
+		</visual>
 	</gazebo>
 	<!-- Cart -->
@@ -61,5 +63,5 @@
 		<origin rpy="0.0 0 0" xyz="0 0 0" />
 		<geometry>
-			<mesh filename="package://meshes/cart-Body.obj" scale="${obj_scale} ${obj_scale} ${obj_scale}" />
+			<mesh filename="$(find cartpole_01)/meshes/cart.dae" scale="${obj_scale} ${obj_scale} ${obj_scale}" />
 		</geometry>
 	</xacro:macro>
@@ -72,11 +74,4 @@
 		<dynamics damping="0.1" />
 	</joint>
-		<gazebo>
-		<plugin filename="libignition-gazebo-apply-joint-force-system.so" name="ignition::gazebo::systems::ApplyJointForce">
-			<joint_name>
-				beam_to_cart
-			</joint_name>
-		</plugin>
-	</gazebo>
 	<link name="cart">
 		<visual>
@@ -93,22 +88,24 @@
 	</link>
 	<gazebo reference="cart">
-		<mu1>
+		<!-- <mu1>
 			0.2
 		</mu1>
 		<mu2>
 			0.2
-		</mu2>
-		<!-- Chrome: http://www.barradeau.com/nicoptere/dump/materials.html -->
-		<material>
-			<diffuse>
-				0.4 0.4 0.4 1
-			</diffuse>
-			<ambient>
-				0.25 0.25 0.25 1
-			</ambient>
-			<specular>
-				0.774597 0.774597 0.774597 1
-			</specular>
-		</material>
+		</mu2> -->
+		<visual>
+			<!-- Chrome: http://www.barradeau.com/nicoptere/dump/materials.html -->
+			<material>
+				<diffuse>
+					0.4 0.4 0.4 1
+				</diffuse>
+				<ambient>
+					0.25 0.25 0.25 1
+				</ambient>
+				<specular>
+					0.774597 0.774597 0.774597 1
+				</specular>
+			</material>
+		</visual>
 	</gazebo>
 	<!-- Pole -->
@@ -116,5 +113,5 @@
 		<origin rpy="0.0 0 0" xyz="0 0 0" />
 		<geometry>
-			<mesh filename="package://meshes/pole-Body.stl" scale="${obj_scale} ${obj_scale} ${obj_scale}" />
+			<mesh filename="$(find cartpole_01)/meshes/pole.dae" scale="${obj_scale} ${obj_scale} ${obj_scale}" />
 		</geometry>
 	</xacro:macro>
@@ -124,14 +121,7 @@
 		<child link="pole" />
 		<limit effort="1000.0" velocity="5.0" />
-		<origin rpy="0 0.01 0" xyz="0 -0.025 0" />
+		<origin rpy="0 -0.5 0" xyz="0 -0.025 0" />
 		<dynamics damping="0.01" />
 	</joint>
-	<gazebo>
-		<plugin filename="libignition-gazebo-apply-joint-force-system.so" name="ignition::gazebo::systems::ApplyJointForce">
-			<joint_name>
-				cart_to_pole
-			</joint_name>
-		</plugin>
-	</gazebo>
 	<link name="pole">
 		<visual>
@@ -148,36 +138,48 @@
 	</link>
 	<gazebo reference="pole">
-		<mu1>
+		<!-- <mu1>
 			0.2
 		</mu1>
 		<mu2>
 			0.2
-		</mu2>
-		<!-- Polished copper: http://www.barradeau.com/nicoptere/dump/materials.html -->
-		<material>
-			<diffuse>
-				<!-- 0.5508 0.2118 0.066 1 -->
-				1 1 1 1
-			</diffuse>
-			<ambient>
-				<!-- 0.2295 0.08825 0.0275 1 -->
-				1 1 1 1
-			</ambient>
-			<specular>
-				<!-- 0.580594 0.223257 0.0695701 1 -->
-				1 1 1 1
-			</specular>
-		</material>
+		</mu2> -->
+		<visual>
+			<!-- Chrome: http://www.barradeau.com/nicoptere/dump/materials.html -->
+			<material>
+				<diffuse>
+					0.4 0.4 0.4 1
+				</diffuse>
+				<ambient>
+					0.25 0.25 0.25 1
+				</ambient>
+				<specular>
+					0.774597 0.774597 0.774597 1
+				</specular>
+			</material>
+		</visual>
 	</gazebo>
 	<!-- Joint states plugin -->
 	<gazebo>
-		<plugin filename="libignition-gazebo-joint-state-publisher-system.so" name="ignition::gazebo::systems::JointStatePublisher">
-			<ros>
-				<remapping>~/out:=joint_states</remapping>
-			</ros>
-	      	<update_rate>30</update_rate>
-		  	<joint_name>beam_to_cart</joint_name>
-		  	<joint_name>cart_to_pole</joint_name>
+	    <!-- <plugin filename="libignition-gazebo-joint-state-publisher-system.so" name="ignition::gazebo::systems::JointStatePublisher"/> -->
+		<!-- <plugin
+			filename="libignition-gazebo-joint-position-controller-system.so"
+			name="ignition::gazebo::systems::JointPositionController">
+				<joint_name>cart_to_pole</joint_name>
+				<p_gain>10</p_gain>
+				<i_gain>1</i_gain>
+				<d_gain>1</d_gain>
+    	</plugin> -->
+		<!-- <plugin
+			filename="libignition-gazebo-physics-system.so"
+			name="ignition::gazebo::systems::Physics">
 		</plugin>
+		<plugin
+			filename="libignition-gazebo-scene-broadcaster-system.so"
+			name="ignition::gazebo::systems::SceneBroadcaster">
+		</plugin>
+		<plugin
+			filename="libignition-gazebo-apply-link-wrench-system.so"
+			name="ignition::gazebo::systems::ApplyLinkWrench">
+		</plugin> -->
 	</gazebo>
 </robot>

Commit message: Fix robot definition and use obj meshes

File: urdf/cartpole.xacro (robot description, xacro)
@@ -2,5 +2,5 @@
 <robot xmlns:xacro="http://www.ros.org/wiki/xacro" name="cartpole">
 	<!-- Properties -->
-	<xacro:property name="obj_scale" value="1.000" />
+	<xacro:property name="obj_scale" value="0.001" />
 	<!-- Define colors -->
 	<material name="black">
@@ -16,5 +16,5 @@
 		<origin rpy="0.0 0 0" xyz="0 0 0" />
 		<geometry>
-			<mesh filename="$(find cartpole_01)/meshes/beam.dae" scale="${obj_scale} ${obj_scale} ${obj_scale}" />
+			<mesh filename="package://meshes/beam-Body.obj" scale="${obj_scale} ${obj_scale} ${obj_scale}" />
 		</geometry>
 	</xacro:macro>
@@ -38,24 +38,22 @@
 	</link>
 	<gazebo reference="beam">
-		<!-- <mu1>
+		<mu1>
 			0.2
 		</mu1>
 		<mu2>
 			0.2
-		</mu2> -->
-		<visual>
-			<!-- Chrome: http://www.barradeau.com/nicoptere/dump/materials.html -->
-			<material>
-				<diffuse>
-					0.4 0.4 0.4 1
-				</diffuse>
-				<ambient>
-					0.25 0.25 0.25 1
-				</ambient>
-				<specular>
-					0.774597 0.774597 0.774597 1
-				</specular>
-			</material>
-		</visual>
+		</mu2>
+		<!-- Chrome: http://www.barradeau.com/nicoptere/dump/materials.html -->
+		<material>
+			<diffuse>
+				0.4 0.4 0.4 1
+			</diffuse>
+			<ambient>
+				0.25 0.25 0.25 1
+			</ambient>
+			<specular>
+				0.774597 0.774597 0.774597 1
+			</specular>
+		</material>
 	</gazebo>
 	<!-- Cart -->
@@ -63,5 +61,5 @@
 		<origin rpy="0.0 0 0" xyz="0 0 0" />
 		<geometry>
-			<mesh filename="$(find cartpole_01)/meshes/cart.dae" scale="${obj_scale} ${obj_scale} ${obj_scale}" />
+			<mesh filename="package://meshes/cart-Body.obj" scale="${obj_scale} ${obj_scale} ${obj_scale}" />
 		</geometry>
 	</xacro:macro>
@@ -74,4 +72,11 @@
 		<dynamics damping="0.1" />
 	</joint>
+		<gazebo>
+		<plugin filename="libignition-gazebo-apply-joint-force-system.so" name="ignition::gazebo::systems::ApplyJointForce">
+			<joint_name>
+				beam_to_cart
+			</joint_name>
+		</plugin>
+	</gazebo>
 	<link name="cart">
 		<visual>
@@ -88,24 +93,22 @@
 	</link>
 	<gazebo reference="cart">
-		<!-- <mu1>
+		<mu1>
 			0.2
 		</mu1>
 		<mu2>
 			0.2
-		</mu2> -->
-		<visual>
-			<!-- Chrome: http://www.barradeau.com/nicoptere/dump/materials.html -->
-			<material>
-				<diffuse>
-					0.4 0.4 0.4 1
-				</diffuse>
-				<ambient>
-					0.25 0.25 0.25 1
-				</ambient>
-				<specular>
-					0.774597 0.774597 0.774597 1
-				</specular>
-			</material>
-		</visual>
+		</mu2>
+		<!-- Chrome: http://www.barradeau.com/nicoptere/dump/materials.html -->
+		<material>
+			<diffuse>
+				0.4 0.4 0.4 1
+			</diffuse>
+			<ambient>
+				0.25 0.25 0.25 1
+			</ambient>
+			<specular>
+				0.774597 0.774597 0.774597 1
+			</specular>
+		</material>
 	</gazebo>
 	<!-- Pole -->
@@ -113,5 +116,5 @@
 		<origin rpy="0.0 0 0" xyz="0 0 0" />
 		<geometry>
-			<mesh filename="$(find cartpole_01)/meshes/pole.dae" scale="${obj_scale} ${obj_scale} ${obj_scale}" />
+			<mesh filename="package://meshes/pole-Body.obj" scale="${obj_scale} ${obj_scale} ${obj_scale}" />
 		</geometry>
 	</xacro:macro>
@@ -121,7 +124,14 @@
 		<child link="pole" />
 		<limit effort="1000.0" velocity="5.0" />
-		<origin rpy="0 -0.5 0" xyz="0 -0.025 0" />
+		<origin rpy="0 0.01 0" xyz="0 -0.025 0" />
 		<dynamics damping="0.01" />
 	</joint>
+	<gazebo>
+		<plugin filename="libignition-gazebo-apply-joint-force-system.so" name="ignition::gazebo::systems::ApplyJointForce">
+			<joint_name>
+				cart_to_pole
+			</joint_name>
+		</plugin>
+	</gazebo>
 	<link name="pole">
 		<visual>
@@ -138,48 +148,36 @@
 	</link>
 	<gazebo reference="pole">
-		<!-- <mu1>
+		<mu1>
 			0.2
 		</mu1>
 		<mu2>
 			0.2
-		</mu2> -->
-		<visual>
-			<!-- Chrome: http://www.barradeau.com/nicoptere/dump/materials.html -->
-			<material>
-				<diffuse>
-					0.4 0.4 0.4 1
-				</diffuse>
-				<ambient>
-					0.25 0.25 0.25 1
-				</ambient>
-				<specular>
-					0.774597 0.774597 0.774597 1
-				</specular>
-			</material>
-		</visual>
+		</mu2>
+		<!-- Polished copper: http://www.barradeau.com/nicoptere/dump/materials.html -->
+		<material>
+			<diffuse>
+				<!-- 0.5508 0.2118 0.066 1 -->
+				1 1 1 1
+			</diffuse>
+			<ambient>
+				<!-- 0.2295 0.08825 0.0275 1 -->
+				1 1 1 1
+			</ambient>
+			<specular>
+				<!-- 0.580594 0.223257 0.0695701 1 -->
+				1 1 1 1
+			</specular>
+		</material>
 	</gazebo>
 	<!-- Joint states plugin -->
 	<gazebo>
-	    <!-- <plugin filename="libignition-gazebo-joint-state-publisher-system.so" name="ignition::gazebo::systems::JointStatePublisher"/> -->
-		<!-- <plugin
-			filename="libignition-gazebo-joint-position-controller-system.so"
-			name="ignition::gazebo::systems::JointPositionController">
-				<joint_name>cart_to_pole</joint_name>
-				<p_gain>10</p_gain>
-				<i_gain>1</i_gain>
-				<d_gain>1</d_gain>
-    	</plugin> -->
-		<!-- <plugin
-			filename="libignition-gazebo-physics-system.so"
-			name="ignition::gazebo::systems::Physics">
+		<plugin filename="libignition-gazebo-joint-state-publisher-system.so" name="ignition::gazebo::systems::JointStatePublisher">
+			<ros>
+				<remapping>~/out:=joint_states</remapping>
+			</ros>
+	      	<update_rate>30</update_rate>
+		  	<joint_name>beam_to_cart</joint_name>
+		  	<joint_name>cart_to_pole</joint_name>
 		</plugin>
-		<plugin
-			filename="libignition-gazebo-scene-broadcaster-system.so"
-			name="ignition::gazebo::systems::SceneBroadcaster">
-		</plugin>
-		<plugin
-			filename="libignition-gazebo-apply-link-wrench-system.so"
-			name="ignition::gazebo::systems::ApplyLinkWrench">
-		</plugin> -->
 	</gazebo>
 </robot>
